Commit message: Port the stack to ROS 2 Humble / Ubuntu 22.04
Upstream targets Jazzy; this machine runs Humble, and the MoveIt Servo API
differs in two ways that only fail at runtime:

- Humble starts Servo with a std_srvs/Trigger on /servo_node/start_servo,
  where Jazzy switches command type via moveit_msgs/ServoCommandType.
- Humble's Servo publishes std_msgs/Int8 on /servo_node/status, not the
  strongly typed moveit_msgs/ServoStatus.

Both launch files select the right API from $ROS_DISTRO at runtime, so the
tree still runs unmodified on Jazzy.

Also:
- servo_params_humble.yaml for the older parameter layout.
- Mesh URIs move from file://$(find pkg) to package://, because
  resource_retriever cannot parse file URLs whose path contains a space,
  and this workspace lives under "Dobot arm".
- setup_dobot.bash sources ROS, the venv and the overlay in one step, and
  presents the install prefixes through a space-free /tmp alias for the
  same reason.
- Ignore .venv/; pin the editor's ROS distro to humble.

Co-Authored-By: Claude Opus 5 (1M context) <noreply@anthropic.com>

File: src/dobot_e6_description/urdf/me6_robot.urdf.xacro (robot description, xacro)
@@ -11,14 +11,14 @@
             <origin xyz="0 0 0" rpy="0 0 0" />
             <geometry>
-                <mesh filename="file://$(find dobot_e6_description)/meshes/me6/base_link.STL" />
-            </geometry>
-            <material name="">
-                <color rgba="0.752941176470588 0.752941176470588 0.752941176470588 1" />
-            </material>
-        </visual>
-        <collision>
-            <origin xyz="0 0 0" rpy="0 0 0" />
-            <geometry>
-                <mesh filename="file://$(find dobot_e6_description)/meshes/me6/base_link.STL" />
+                <mesh filename="package://dobot_e6_description/meshes/me6/base_link.STL" />
+            </geometry>
+            <material name="">
+                <color rgba="0.752941176470588 0.752941176470588 0.752941176470588 1" />
+            </material>
+        </visual>
+        <collision>
+            <origin xyz="0 0 0" rpy="0 0 0" />
+            <geometry>
+                <mesh filename="package://dobot_e6_description/meshes/me6/base_link.STL" />
             </geometry>
         </collision>
@@ -43,14 +43,14 @@
             <origin xyz="0 0 0" rpy="0 0 0" />
             <geometry>
-                <mesh filename="file://$(find dobot_e6_description)/meshes/me6/Link1.STL" />
-            </geometry>
-            <material name="">
-                <color rgba="0.752941176470588 0.752941176470588 0.752941176470588 1" />
-            </material>
-        </visual>
-        <collision>
-            <origin xyz="0 0 0" rpy="0 0 0" />
-            <geometry>
-                <mesh filename="file://$(find dobot_e6_description)/meshes/me6/Link1.STL" />
+                <mesh filename="package://dobot_e6_description/meshes/me6/Link1.STL" />
+            </geometry>
+            <material name="">
+                <color rgba="0.752941176470588 0.752941176470588 0.752941176470588 1" />
+            </material>
+        </visual>
+        <collision>
+            <origin xyz="0 0 0" rpy="0 0 0" />
+            <geometry>
+                <mesh filename="package://dobot_e6_description/meshes/me6/Link1.STL" />
             </geometry>
         </collision>
@@ -72,14 +72,14 @@
             <origin xyz="0 0 0" rpy="0 0 0" />
             <geometry>
-                <mesh filename="file://$(find dobot_e6_description)/meshes/me6/Link2.STL" />
-            </geometry>
-            <material name="">
-                <color rgba="0.752941176470588 0.752941176470588 0.752941176470588 1" />
-            </material>
-        </visual>
-        <collision>
-            <origin xyz="0 0 0" rpy="0 0 0" />
-            <geometry>
-                <mesh filename="file://$(find dobot_e6_description)/meshes/me6/Link2.STL" />
+                <mesh filename="package://dobot_e6_description/meshes/me6/Link2.STL" />
+            </geometry>
+            <material name="">
+                <color rgba="0.752941176470588 0.752941176470588 0.752941176470588 1" />
+            </material>
+        </visual>
+        <collision>
+            <origin xyz="0 0 0" rpy="0 0 0" />
+            <geometry>
+                <mesh filename="package://dobot_e6_description/meshes/me6/Link2.STL" />
             </geometry>
         </collision>
@@ -101,14 +101,14 @@
             <origin xyz="0 0 0" rpy="0 0 0" />
             <geometry>
-                <mesh filename="file://$(find dobot_e6_description)/meshes/me6/Link3.STL" />
-            </geometry>
-            <material name="">
-                <color rgba="0.752941176470588 0.752941176470588 0.752941176470588 1" />
-            </material>
-        </visual>
-        <collision>
-            <origin xyz="0 0 0" rpy="0 0 0" />
-            <geometry>
-                <mesh filename="file://$(find dobot_e6_description)/meshes/me6/Link3.STL" />
+                <mesh filename="package://dobot_e6_description/meshes/me6/Link3.STL" />
+            </geometry>
+            <material name="">
+                <color rgba="0.752941176470588 0.752941176470588 0.752941176470588 1" />
+            </material>
+        </visual>
+        <collision>
+            <origin xyz="0 0 0" rpy="0 0 0" />
+            <geometry>
+                <mesh filename="package://dobot_e6_description/meshes/me6/Link3.STL" />
             </geometry>
         </collision>
@@ -130,14 +130,14 @@
             <origin xyz="0 0 0" rpy="0 0 0" />
             <geometry>
-                <mesh filename="file://$(find dobot_e6_description)/meshes/me6/Link4.STL" />
-            </geometry>
-            <material name="">
-                <color rgba="0.752941176470588 0.752941176470588 0.752941176470588 1" />
-            </material>
-        </visual>
-        <collision>
-            <origin xyz="0 0 0" rpy="0 0 0" />
-            <geometry>
-                <mesh filename="file://$(find dobot_e6_description)/meshes/me6/Link4.STL" />
+                <mesh filename="package://dobot_e6_description/meshes/me6/Link4.STL" />
+            </geometry>
+            <material name="">
+                <color rgba="0.752941176470588 0.752941176470588 0.752941176470588 1" />
+            </material>
+        </visual>
+        <collision>
+            <origin xyz="0 0 0" rpy="0 0 0" />
+            <geometry>
+                <mesh filename="package://dobot_e6_description/meshes/me6/Link4.STL" />
             </geometry>
         </collision>
@@ -159,14 +159,14 @@
             <origin xyz="0 0 0" rpy="0 0 0" />
             <geometry>
-                <mesh filename="file://$(find dobot_e6_description)/meshes/me6/Link5.STL" />
-            </geometry>
-            <material name="">
-                <color rgba="0.752941176470588 0.752941176470588 0.752941176470588 1" />
-            </material>
-        </visual>
-        <collision>
-            <origin xyz="0 0 0" rpy="0 0 0" />
-            <geometry>
-                <mesh filename="file://$(find dobot_e6_description)/meshes/me6/Link5.STL" />
+                <mesh filename="package://dobot_e6_description/meshes/me6/Link5.STL" />
+            </geometry>
+            <material name="">
+                <color rgba="0.752941176470588 0.752941176470588 0.752941176470588 1" />
+            </material>
+        </visual>
+        <collision>
+            <origin xyz="0 0 0" rpy="0 0 0" />
+            <geometry>
+                <mesh filename="package://dobot_e6_description/meshes/me6/Link5.STL" />
             </geometry>
         </collision>
@@ -188,5 +188,5 @@
             <origin xyz="0 0 0" rpy="0 0 0" />
             <geometry>
-                <mesh filename="file://$(find dobot_e6_description)/meshes/me6/Link6.STL" />
+                <mesh filename="package://dobot_e6_description/meshes/me6/Link6.STL" />
             </geometry>
             <material name="">
@@ -197,5 +197,5 @@
             <origin xyz="0 0 0" rpy="0 0 0" />
             <geometry>
-                <mesh filename="file://$(find dobot_e6_description)/meshes/me6/Link6.STL" />
+                <mesh filename="package://dobot_e6_description/meshes/me6/Link6.STL" />
             </geometry>
         </collision>
