Commit message: Pivot teleop rotations on the probe instead of the flange
MoveIt Servo computes its Jacobian at the tip of its group chain, and that
chain ended at Link6 -- so roll, pitch and yaw all turned about the bare
flange. A new fixed frame, probe_tcp, sits at (-65, 0, 98) mm from the flange
and the Servo chain now ends there (ee_frame_name too), so rotations pivot on
the probe and translations move that point.

Checked offline: Servo run against an arm held at home, pure rotation commands
about each axis. The flange moved 0.26-0.47 mm per step while probe_tcp moved
0.000-0.001 mm. The condition number at home barely changes (15.92 -> 16.14),
so the singularity thresholds behave as before.

The Windows teleop streams Cartesian poses of the robot's own tool frame, so it
sets tool 1 to the same offset and selects it. Haptics compute kappa at the same
point Servo uses.

The test also caught an XML comment containing "--", which would have stopped
the robot model loading at launch.

Not yet run on the arm.

Co-Authored-By: Claude Opus 5.5 <noreply@anthropic.com>

File: src/dobot_e6_bringup/robots/probe_wrapper_e6.urdf.xacro (robot description, xacro)
@@ -10,4 +10,11 @@
   <xacro:arg name="simulation_controllers" default="" />
   <xacro:arg name="initial_positions_file" default="" />
+  <!-- Tool centre point: where teleop rotations pivot and translations are
+       measured. Offset from the flange (Link6) in metres, Link6 frame.
+       Currently the probe assembly's centre of mass (-65, 0, 98) mm; move it
+       to the probe tip if that is where rotations should pivot. -->
+  <xacro:arg name="tcp_x" default="-0.065" />
+  <xacro:arg name="tcp_y" default="0.0" />
+  <xacro:arg name="tcp_z" default="0.098" />
   <xacro:property name="initial_positions"
                   value="${xacro.load_yaml('$(arg initial_positions_file)')}" />
@@ -37,4 +44,13 @@
     </inertial>
   </link>
+  <!-- Tool centre point. MoveIt Servo's chain ends here (servo_moveit_params.yaml),
+       so its Jacobian, and therefore every teleop rotation, is about this point, not
+       the bare flange. -->
+  <link name="probe_tcp" />
+  <joint name="probe_tcp_joint" type="fixed">
+    <parent link="Link6" />
+    <child link="probe_tcp" />
+    <origin xyz="$(arg tcp_x) $(arg tcp_y) $(arg tcp_z)" rpy="0 0 0" />
+  </joint>
   <!-- FIXED joint to the flange. The FT sensor reads the wrench through it. -->
   <joint name="us_probe_joint" type="fixed">
